File: mmWave-radarBoard/FTDI.kicad_sch (KiCad schematic)
At the start: 42 parts, among them U301 FT4232HQ, U302 93LCxxB, Y301 12MHz

Commit message: Updated schematic and layout PCB
Parts:
- renumbered C301 to C64, C302 to C65, C303 to C66, C304 to C67, C305 to C68, C306 to C69, C307 to C70, C308 to C71, C309 to C72, C310 to C73, C311 to C74, C312 to C75, C313 to C76, C314 to C77, C315 to C78, C316 to C79, D301 to D7, FB301 to FB5, FB302 to FB6, FB303 to FB7, R301 to R28, R302 to R29, R303 to R30, R304 to R31, R305 to R32, R306 to R33, R307 to R34, R308 to R35, R309 to R36, R310 to R37, R311 to R38, R312 to R39, R313 to R40, R314 to R41, R315 to R42, R316 to R43, R317 to R44, R318 to R45, R319 to R46, U301 to U7, U302 to U8, Y301 to Y1
Other:
- title: FTDI -> Power
