File: mmWave-radarBoard/Power.kicad_sch (KiCad schematic)
At the start: 122 parts, among them J201 Conn_01x02_Socket, J203 USB4120-03-C, Q201 BSS123, U201 TPS628502DRLR, U202 USBLC6-2P6, U203 TPS628502DRLR, U204 TPS2116DRL, U205 XI6432BRQAAMY, U206 TLV75533PDRV

Commit message: Updated PCB
Parts:
- R201, R202, R205, R206, R211, R212, R213, R214, R215, R216, R217, R221, R222, R223, R224, R225: footprint Resistor_SMD:R_0201_0603Metric -> Resistor_SMD:R_0402_1005Metric
Changed lines of the file:
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@@
 			)
 		)
-		(property "Footprint" "Resistor_SMD:R_0201_0603Metric"
+		(property "Footprint" "Resistor_SMD:R_0402_1005Metric"
 			(at 372.11 85.598 90)
 			(effects
@@
 			)
 		)
-		(property "Footprint" "Resistor_SMD:R_0201_0603Metric"
+		(property "Footprint" "Resistor_SMD:R_0402_1005Metric"
 			(at 112.268 279.4 90)
 			(effects
@@
 			)
 		)
-		(property "Footprint" "Resistor_SMD:R_0201_0603Metric"
+		(property "Footprint" "Resistor_SMD:R_0402_1005Metric"
 			(at 440.182 99.06 90)
 			(effects
@@
 			)
 		)
-		(property "Footprint" "Resistor_SMD:R_0201_0603Metric"
+		(property "Footprint" "Resistor_SMD:R_0402_1005Metric"
 			(at 372.872 96.52 90)
 			(effects
@@
 			)
 		)
-		(property "Footprint" "Resistor_SMD:R_0201_0603Metric"
+		(property "Footprint" "Resistor_SMD:R_0402_1005Metric"
 			(at 372.872 172.72 90)
 			(effects
@@
 			)
 		)
-		(property "Footprint" "Resistor_SMD:R_0201_0603Metric"
+		(property "Footprint" "Resistor_SMD:R_0402_1005Metric"
 			(at 372.11 161.798 90)
 			(effects
@@
 			)
 		)
-		(property "Footprint" "Resistor_SMD:R_0201_0603Metric"
+		(property "Footprint" "Resistor_SMD:R_0402_1005Metric"
 			(at 440.182 83.82 90)
 			(effects
@@
 			)
 		)
-		(property "Footprint" "Resistor_SMD:R_0201_0603Metric"
+		(property "Footprint" "Resistor_SMD:R_0402_1005Metric"
 			(at 43.942 190.5 90)
 			(effects
@@
 			)
 		)
-		(property "Footprint" "Resistor_SMD:R_0201_0603Metric"
+		(property "Footprint" "Resistor_SMD:R_0402_1005Metric"
 			(at 142.748 191.77 90)
 			(effects
@@
 			)
 		)
-		(property "Footprint" "Resistor_SMD:R_0201_0603Metric"
+		(property "Footprint" "Resistor_SMD:R_0402_1005Metric"
 			(at 124.46 253.238 90)
 			(effects
@@
 			)
 		)
-		(property "Footprint" "Resistor_SMD:R_0201_0603Metric"
+		(property "Footprint" "Resistor_SMD:R_0402_1005Metric"
 			(at 43.942 177.8 90)
 			(effects
@@
 			)
 		)
-		(property "Footprint" "Resistor_SMD:R_0201_0603Metric"
+		(property "Footprint" "Resistor_SMD:R_0402_1005Metric"
 			(at 104.14 272.288 90)
 			(effects
@@
 			)
 		)
-		(property "Footprint" "Resistor_SMD:R_0201_0603Metric"
+		(property "Footprint" "Resistor_SMD:R_0402_1005Metric"
 			(at 104.14 253.238 90)
 			(effects
@@
 			)
 		)
-		(property "Footprint" "Resistor_SMD:R_0201_0603Metric"
+		(property "Footprint" "Resistor_SMD:R_0402_1005Metric"
 			(at 440.182 160.02 90)
 			(effects
@@
 			)
 		)
-		(property "Footprint" "Resistor_SMD:R_0201_0603Metric"
+		(property "Footprint" "Resistor_SMD:R_0402_1005Metric"
 			(at 74.93 291.338 90)
 			(effects
@@
 			)
 		)
-		(property "Footprint" "Resistor_SMD:R_0201_0603Metric"
+		(property "Footprint" "Resistor_SMD:R_0402_1005Metric"
 			(at 440.182 175.26 90)
 			(effects

Commit message: Updated PCB
Parts:
- removed J201: Conn_01x02_Socket, Connector_JST:JST_ZH_B2B-ZR_1x02_P1.50mm_Vertical, symbol Connector:Conn_01x02_Socket
- added J104: Conn_01x03_Socket, Connector_JST:JST_ZE_B03B-ZESK-D_1x03_P1.50mm_Vertical, symbol Connector:Conn_01x03_Socket
Connections:
- net GND: now also J104.1 (Pin_1), J104.2 (Pin_2)
- net at F201.1: now also J104.3 (Pin_3)
Changed lines of the file:
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@@
 	(text "5V 3A"
 		(exclude_from_sim no)
-		(at 228.6 86.36 0)
+		(at 228.6 88.9 0)
 		(effects
 			(font
@@
 	)
 	(junction
+		(at 233.68 85.09)
+		(diameter 0)
+		(color 0 0 0 0)
+	)
+	(junction
 		(at 532.13 322.58)
 		(diameter 0)
@@
 	(wire
 		(pts
+			(xy 233.68 85.09) (xy 233.68 92.71)
+		)
+		(stroke
+			(width 0)
+			(type default)
+		)
+	)
+	(wire
+		(pts
 			(xy 73.66 90.17) (xy 77.47 90.17)
 		)
@@
 	(wire
 		(pts
-			(xy 233.68 82.55) (xy 233.68 92.71)
+			(xy 233.68 82.55) (xy 233.68 85.09)
 		)
 		(stroke
@@
 	(wire
 		(pts
+			(xy 231.14 85.09) (xy 233.68 85.09)
+		)
+		(stroke
+			(width 0)
+			(type default)
+		)
+	)
+	(wire
+		(pts
 			(xy 523.24 115.57) (xy 528.32 115.57)
 		)
@@
 	)
 	(symbol
-		(lib_id "Connector:Conn_01x02_Socket")
-		(at 226.06 80.01 0)
-		(mirror y)
-		(unit 1)
-		(exclude_from_sim no)
-		(in_bom yes)
-		(on_board yes)
-		(dnp no)
-		(fields_autoplaced yes)
-		(property "Reference" "J201"
-			(at 226.695 74.93 0)
-			(effects
-				(font
-					(size 1.27 1.27)
-				)
-			)
-		)
-		(property "Value" "Conn_01x02_Socket"
-			(at 226.695 77.47 0)
-			(effects
-				(font
-					(size 1.27 1.27)
-				)
-			)
-		)
-		(property "Footprint" "Connector_JST:JST_ZH_B2B-ZR_1x02_P1.50mm_Vertical"
-			(at 226.06 80.01 0)
-			(effects
-				(font
-					(size 1.27 1.27)
-				)
-				(hide yes)
-			)
-		)
-		(property "Datasheet" "~"
-			(at 226.06 80.01 0)
-			(effects
-				(font
-					(size 1.27 1.27)
-				)
-				(hide yes)
-			)
-		)
-		(property "Description" "Generic connector, single row, 01x02, script generated"
-			(at 226.06 80.01 0)
-			(effects
-				(font
-					(size 1.27 1.27)
-				)
-				(hide yes)
-			)
-		)
-		(pin "1"
-		)
-		(pin "2"
-		)
-		(instances
-			(project ""
-				(path "/65d1bf45-0c7d-403c-8da5-e1777d98e937/63e9aa23-19c0-43a2-8100-8d16d5100cb9"
-					(reference "J201")
-					(unit 1)
-				)
-			)
-		)
-	)
-	(symbol
 		(lib_id "Device:C")
 		(at 325.12 83.82 0)
@@
 					(unit 1)
 				)
+			)
+		)
+	)
+	(symbol
+		(lib_id "Connector:Conn_01x03_Socket")
+		(at 226.06 82.55 180)
+		(unit 1)
+		(exclude_from_sim no)
+		(in_bom yes)
+		(on_board yes)
+		(dnp no)
+		(property "Reference" "J104"
+			(at 224.79 83.8201 0)
+			(effects
+				(font
+					(size 1.27 1.27)
+				)
+				(justify left)
+			)
+		)
+		(property "Value" "Conn_01x03_Socket"
+			(at 224.79 81.2801 0)
+			(effects
+				(font
+					(size 1.27 1.27)
+				)
+				(justify left)
+				(hide yes)
+			)
+		)
+		(property "Footprint" "Connector_JST:JST_ZE_B03B-ZESK-D_1x03_P1.50mm_Vertical"
+			(at 226.06 82.55 0)
+			(effects
+				(font
+					(size 1.27 1.27)
+				)
+				(hide yes)
+			)
+		)
+		(property "Datasheet" "~"
+			(at 226.06 82.55 0)
+			(effects
+				(font
+					(size 1.27 1.27)
+				)
+				(hide yes)
+			)
+		)
+		(property "Description" "Generic connector, single row, 01x03, script generated"
+			(at 226.06 82.55 0)
+			(effects
+				(font
+					(size 1.27 1.27)
+				)
+				(hide yes)
+			)
+		)
+		(pin "3"
+		)
+		(pin "2"
+		)
+		(pin "1"
+		)
+		(instances
+			(project "mmWave-radarBoard"
+				(path "/65d1bf45-0c7d-403c-8da5-e1777d98e937/63e9aa23-19c0-43a2-8100-8d16d5100cb9"
+					(reference "J104")
+					(unit 1)
+				)

Commit message: Updated schematic and layout PCB
Parts:
- Q2: renamed from MOSFET201; footprint SSM3K35AMFV:VESM_TOS-L -> SSM3K35AMFV:VESM_TOS-M
- renumbered C201 to C1, C210 to C10, C211 to C11, C212 to C12, C213 to C13, C214 to C14, C215 to C15, C216 to C16, C217 to C17, C218 to C18, C219 to C19, C202 to C2, C220 to C20, C221 to C21, C222 to C22, C223 to C23, C224 to C24, C225 to C25, C226 to C26, C227 to C27, C228 to C28, C229 to C29, C203 to C3, C230 to C30, C231 to C31, C232 to C32, C233 to C33, C234 to C34, C235 to C35, C236 to C36, C237 to C37, C238 to C38, C239 to C39, C204 to C4, C240 to C40, C241 to C41, C242 to C42, C243 to C43, C244 to C44, C245 to C45, C246 to C46, C247 to C47, C248 to C48, C249 to C49, C205 to C5, C250 to C50, C251 to C51, C252 to C52, C253 to C53, C254 to C54, C255 to C55, C256 to C56, C257 to C57, C258 to C58, C259 to C59, C206 to C6, C260 to C60, C261 to C61, C262 to C62, C263 to C63, C207 to C7, C208 to C8, C209 to C9, D201 to D1, D202 to D2, D203 to D3, D204 to D4, D205 to D5, D206 to D6, F201 to F1, FB201 to FB1, FB202 to FB2, FB203 to FB3, FB204 to FB4, J104 to J4, J203 to J5, L201 to L1, L202 to L2, L203 to L3, L204 to L4, L205 to L5, Q201 to Q1, R208 to R10, R209 to R11, R210 to R12, R211 to R13, R212 to R14, R213 to R15, R214 to R16, R215 to R17, R216 to R18, R217 to R19, R218 to R20, R219 to R21, R220 to R22, R221 to R23, R222 to R24, R223 to R25, R224 to R26, R225 to R27, R201 to R3, R202 to R4, R203 to R5, R204 to R6, R205 to R7, R206 to R8, R207 to R9, TP201 to TP1, TP202 to TP2, TP203 to TP3, TP204 to TP4, TP205 to TP5, TP206 to TP6, TP207 to TP7, TP208 to TP8, U201 to U1, U202 to U2, U203 to U3, U204 to U4, U205 to U5, U206 to U6
