File: mmWave-radarBoard/mmWave-radarBoard.kicad_pcb (KiCad board)
At the start: 6 copper layers, 55 x 84.1 mm, 276 parts, among them J1 Conn_01x07_Socket, J2 Conn_01x03_Socket, J3 Conn_01x06_Socket, J4 Conn_01x03_Socket, J5 USB4120-03-C, J6 Conn_01x03_Socket, J7 Conn_01x03_Socket, J8 Conn_01x03_Socket, J9 Conn_02x06_Odd_Even, Q1 BSS123, Q2 SSM3K35AMFV_L3F, Q3 SSM3K35AMFV_L3F, Q4 SSM3K35AMFV_L3F, SW1 SW_DPST, SW2 SW_DPST, SW3 SW_SPDT, SW4 SW_DIP_x04, U1 TPS628502DRLR, U10 TLIN1039DDFRQ1, U11 TRS3221EIDBR, U12 MX25R1635FZUIH0, U13 TS3A5018RSVR, U14 SN74LVC1G11DSFR, U2 USBLC6-2P6, U3 TPS628502DRLR, U4 TPS2116DRL, U5 XI6432BRQAAMY, U6 TLV75533PDRV, U7 FT4232HQ, U8 93LCxxB, U9 TCAN1042HGVDRQ1, Y1 12MHz, Y2 40MHz

Commit message: Started routing
Parts:
- removed TP12: TestPoint, TestPoint:TestPoint_Pad_D1.0mm
- moved TP4 4.40 mm to (146.2, 84.9)
- moved TP3 2.23 mm to (141.8, 84.9)
- turned R22 to 90 degrees
Routing:
- net VCC_3V3: track 21.0 -> 227.3 mm, vias 1 -> 11
- net 5V_IN: track 17.7 -> 122.8 mm, vias 0 -> 6
- net FTDI_3V3: track 11.7 -> 78.2 mm, vias 0 -> 5
- net /RADAR_~{RST}: track 2.95 -> 66.3 mm
- net /TDO_SOP0: track 0.00 -> 42.5 mm
- net /REG_MODE_SELECT: track 0.00 -> 38.9 mm
- net /SPI_CS_I2C_SDA: track 1.04 -> 38.4 mm
- net /HOST_INTR_GPIO_0_LED: track 0.32 -> 37.1 mm
- net /TMS: track 0.35 -> 34.1 mm
- net /Power/REG_PG: track 1.66 -> 29.9 mm, vias 2 -> 3
- net /SPI_CLK_I2C_SCL: track 1.07 -> 29.0 mm, vias 0 -> 1
- net FTDI_VCORE: track 6.44 -> 33.8 mm, vias 0 -> 4
- net /RS232_TX: track 2.37 -> 29.2 mm
- net /RS232_RX: track 3.04 -> 28.8 mm
- net /SPI_MISO_REG_MODE: track 0.32 -> 25.9 mm, vias 1 -> 2
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