File: mmWave-radarBoard/Muxes.kicad_sch (KiCad schematic)
At the start: 38 parts, among them SW601 SW_DPST, SW602 SW_DPST, SW603 SW_SPDT, SW604 SW_DIP_x04, U601 TS3A5018RSVR, U602 SN74LVC1G11DSFR

Commit message: Updated schematic and layout PCB
Parts:
- Q3: renamed from MOSFET601; footprint SSM3K35AMFV:VESM_TOS-L -> SSM3K35AMFV:VESM_TOS-M
- Q4: renamed from MOSFET602; footprint SSM3K35AMFV:VESM_TOS-L -> SSM3K35AMFV:VESM_TOS-M
- renumbered C601 to C97, C602 to C98, C603 to C99, D601 to D11, D602 to D12, R624 to R100, R601 to R77, R602 to R78, R603 to R79, R604 to R80, R605 to R81, R606 to R82, R607 to R83, R608 to R84, R609 to R85, R610 to R86, R611 to R87, R612 to R88, R613 to R89, R614 to R90, R615 to R91, R616 to R92, R617 to R93, R618 to R94, R619 to R95, R620 to R96, R621 to R97, R622 to R98, R623 to R99, SW601 to SW1, SW602 to SW2, SW603 to SW3, SW604 to SW4, TP601 to TP15, U601 to U13, U602 to U14
Connections:
- net at SW2.1, SW2.3: now also R88.2, R89.2; no longer R86.1
- net at SW2.2, SW2.4: now also R86.1; no longer R88.2, R89.2
Other:
- title: Muxes -> Power
