File: mmWave-radarBoard/mmWave-radarBoard.kicad_sch (KiCad schematic)
At the start: 7 parts, among them J101 Conn_01x03_Socket, J102 Conn_01x07_Socket, J103 Conn_01x06_Socket

Commit message: Updated PCB
Parts:
- added R320, R321: 4.7k, Resistor_SMD:R_0402_1005Metric, symbol Device:R
Connections:
- net I2C_SCL: now also R320.1
- net I2C_SDA: now also R321.1
- net VCC_3V3: now also R320.2, R321.2
Other:
- moved on the sheet: J101

Commit message: Updated schematic and layout PCB
Parts:
- renumbered H101 to H1, H102 to H2, H103 to H3, H104 to H4, J102 to J1, J101 to J2, J103 to J3, R320 to R1, R321 to R2
Connections:
- net GND: now also J2.1 (Pin_1); no longer J2.3 (Pin_3)
- net I2C_SCL: now also J2.3 (Pin_3); no longer J2.1 (Pin_1)
Other:
- title: Main -> Power
- moved on the sheet: J1, J3
