File: mmWave-radarBoard/xWRL6432AOP_interface.kicad_sch (KiCad schematic)
At the start: 35 parts, among them J9 Conn_02x06_Odd_Even, U12 MX25R1635FZUIH0, U5 XI6432BRQAAMY, Y2 40MHz

Commit message: Started routing
Parts:
- removed TP12: TestPoint, TestPoint:TestPoint_Pad_D1.0mm, symbol Connector:TestPoint
Changed lines of the file:
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@@
 	)
 	(junction
-		(at 140.97 44.45)
-		(diameter 0)
-		(color 0 0 0 0)
-	)
-	(junction
 		(at 120.65 125.73)
 		(diameter 0)
@@
 	(wire
 		(pts
-			(xy 140.97 44.45) (xy 140.97 45.72)
+			(xy 140.97 43.18) (xy 140.97 44.45)
 		)
 		(stroke
@@
 	(wire
 		(pts
-			(xy 135.89 44.45) (xy 140.97 44.45)
-		)
-		(stroke
-			(width 0)
-			(type default)
-		)
-	)
-	(wire
-		(pts
 			(xy 69.85 124.46) (xy 72.39 124.46)
 		)
@@
 	(wire
 		(pts
-			(xy 140.97 43.18) (xy 140.97 44.45)
-		)
-		(stroke
-			(width 0)
-			(type default)
-		)
-	)
-	(wire
-		(pts
 			(xy 57.15 132.08) (xy 54.61 132.08)
 		)
@@
 	(symbol
 		(lib_id "power:GND")
-		(at 140.97 45.72 0)
+		(at 140.97 44.45 0)
 		(unit 1)
 		(exclude_from_sim no)
@@
 		(fields_autoplaced yes)
 		(property "Reference" "#PWR0171"
-			(at 140.97 52.07 0)
+			(at 140.97 50.8 0)
 			(effects
 				(font
@@
 		)
 		(property "Value" "GND"
-			(at 140.97 50.8 0)
+			(at 140.97 49.53 0)
 			(effects
 				(font
@@
 		)
 		(property "Footprint" ""
-			(at 140.97 45.72 0)
+			(at 140.97 44.45 0)
 			(effects
 				(font
@@
 		)
 		(property "Datasheet" ""
-			(at 140.97 45.72 0)
+			(at 140.97 44.45 0)
 			(effects
 				(font
@@
 		)
 		(property "Description" "Power symbol creates a global label with name \"GND\" , ground"
-			(at 140.97 45.72 0)
+			(at 140.97 44.45 0)
 			(effects
 				(font
@@
 					(unit 1)
 				)
-			)
-		)
-	)
-	(symbol
-		(lib_id "Connector:TestPoint")
-		(at 135.89 44.45 90)
-		(unit 1)
-		(exclude_from_sim no)
-		(in_bom yes)
-		(on_board yes)
-		(dnp no)
-		(fields_autoplaced yes)
-		(property "Reference" "TP12"
-			(at 132.588 39.37 90)
-			(effects
-				(font
-					(size 1.27 1.27)
-				)
-			)
-		)
-		(property "Value" "TestPoint"
-			(at 132.588 41.91 90)
-			(effects
-				(font
-					(size 1.27 1.27)
-				)
-			)
-		)
-		(property "Footprint" "TestPoint:TestPoint_Pad_D1.0mm"
-			(at 135.89 39.37 0)
-			(effects
-				(font
-					(size 1.27 1.27)
-				)
-				(hide yes)
-			)
-		)
-		(property "Datasheet" "~"
-			(at 135.89 39.37 0)
-			(effects
-				(font
-					(size 1.27 1.27)
-				)
-				(hide yes)
-			)
-		)
-		(property "Description" "test point"
-			(at 135.89 44.45 0)
-			(effects
-				(font
-					(size 1.27 1.27)
-				)
-				(hide yes)
-			)
-		)
-		(pin "1"
-		)
-		(instances
-			(project "mmWave-radarBoard"
-				(path "/65d1bf45-0c7d-403c-8da5-e1777d98e937/67383843-b151-490b-b925-303d04bb18ba"
-					(reference "TP12")
-					(unit 1)
-				)
